File: Schematics/OurStuff/ECE477/ECE477.kicad_sch (KiCad schematic)
At the start: 65 parts, among them J1 USB_B_Micro, J2 Barrel_Jack, J3 OLED JST PH 7pin, J7 D30V30F3, Q1 SS8050-G, Q2 SS8050-G, U1 ESP32-WROOM-32E, U2 CP2102N-Axx-xQFN28, U3 USBLC6-2SC6

Commit message: added power label
Changed lines of the file:
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@@
 	(title_block
 		(title "ECE477 Translating Glasses")
-		(date "2025-02-18")
+		(date "2025-03-12")
 	)
 	(junction
@@
 	)
 	(junction
+		(at 149.86 107.95)
+		(diameter 0)
+		(color 0 0 0 0)
+	)
+	(junction
 		(at 359.41 29.21)
 		(diameter 0)
@@
 	(wire
 		(pts
+			(xy 149.86 107.95) (xy 149.86 110.49)
+		)
+		(stroke
+			(width 0)
+			(type default)
+		)
+	)
+	(wire
+		(pts
 			(xy 240.03 226.06) (xy 240.03 229.87)
 		)
@@
 	(wire
 		(pts
-			(xy 149.86 105.41) (xy 149.86 110.49)
+			(xy 149.86 105.41) (xy 149.86 107.95)
 		)
 		(stroke
@@
 					(unit 1)
 				)
+			)
+		)
+	)
+	(symbol
+		(lib_id "power:PWR_FLAG")
+		(at 149.86 107.95 270)
+		(unit 1)
+		(exclude_from_sim no)
+		(in_bom yes)
+		(on_board yes)
+		(dnp no)
+		(fields_autoplaced yes)
+		(property "Reference" "#FLG02"
+			(at 151.765 107.95 0)
+			(effects
+				(font
+					(size 1.27 1.27)
+				)
+				(hide yes)
+			)
+		)
+		(property "Value" "PWR_FLAG"
+			(at 153.67 107.9499 90)
+			(effects
+				(font
+					(size 1.27 1.27)
+				)
+				(justify left)
+			)
+		)
+		(property "Footprint" ""
+			(at 149.86 107.95 0)
+			(effects
+				(font
+					(size 1.27 1.27)
+				)
+				(hide yes)
+			)
+		)
+		(property "Datasheet" "~"
+			(at 149.86 107.95 0)
+			(effects
+				(font
+					(size 1.27 1.27)
+				)
+				(hide yes)
+			)
+		)
+		(property "Description" "Special symbol for telling ERC where power comes from"
+			(at 149.86 107.95 0)
+			(effects
+				(font
+					(size 1.27 1.27)
+				)
+				(hide yes)
+			)
+		)
+		(pin "1"
+		)
+		(instances
+			(project "ECE477"
+				(path "/f5b3def7-e561-4cb3-8a45-4eba76d025b6"
+					(reference "#FLG02")
+					(unit 1)
+				)

Commit message: updated PCB with suggestions 1-4
Parts:
- R3: value 2k -> 1k
Changed lines of the file:
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@@
 			)
 		)
-		(property "Value" "2k"
+		(property "Value" "1k"
 			(at 218.44 161.29 90)
 			(effects
